Commit message: feat: add scene3 implementation, camera view, data collection
- Add scene3_impl.py with tray detection logic
- Add camera_view.py for camera visualization
- Add collect_data.py for data gathering
- Add train_yolo.py and data.yaml for YOLO training pipeline
- Update URDF and XML model files for biped_s52
- Update challenge_task.py
- Add CLAUDE.md and agent docs
- Add .gitignore rules for model weights and training data

Co-Authored-By: Claude Opus 4.8 <noreply@anthropic.com>

File: src/kuavo_assets/models/biped_s52/urdf/biped_s52.urdf (robot description, URDF)
Before this commit: robot biped_s52, 48 links, 47 joints
Links:
- link waist_yaw_link: mass 19.54016 -> 16.28826

File: src/kuavo_assets/models/biped_s52/urdf/biped_s52_gazebo.urdf (robot description, URDF)
Before this commit: robot biped_s52, 48 links, 47 joints
Links:
- link waist_yaw_link: mass 19.54016 -> 16.28826

File: src/kuavo_assets/models/biped_s52/urdf/drake/biped_v3.urdf (robot description, URDF)
Before this commit: robot biped_v3, 14 links, 13 joints
Links:
- link waist_yaw_link: mass 32.44746 -> 29.19556

File: src/kuavo_assets/models/biped_s52/urdf/drake/biped_v3_all_joint.urdf (robot description, URDF)
Before this commit: robot biped_v3_all_joint, 35 links, 30 joints
Links:
- link torso: mass 37.32594316 -> 34.07404316

File: src/kuavo_assets/models/biped_s52/urdf/drake/biped_v3_full.urdf (robot description, URDF)
Before this commit: robot biped_s52, 32 links, 31 joints
Links:
- link waist_yaw_link: mass 21.46335568 -> 18.21145568

Commit message: feat: add scene3 implementation, camera view, data collection
- Add scene3_impl.py with tray detection logic
- Add camera_view.py for camera visualization
- Add collect_data.py for data gathering
- Add train_yolo.py and data.yaml for YOLO training pipeline
- Update URDF and XML model files for biped_s52
- Update challenge_task.py
- Add CLAUDE.md and agent docs
- Add .gitignore rules for model weights and training data

Co-Authored-By: Claude Opus 4.8 <noreply@anthropic.com>


Revert commit: feat: add scene3 implementation, camera view, data collection
This revert commit: 33f8f77062f1f2ff591e9c4540243d924bbfec04

File: src/kuavo_assets/models/biped_s52/urdf/biped_s52.urdf (robot description, URDF)
Before this commit: robot biped_s52, 48 links, 47 joints
Links:
- link waist_yaw_link: mass 16.28826 -> 19.54016

File: src/kuavo_assets/models/biped_s52/urdf/biped_s52_gazebo.urdf (robot description, URDF)
Before this commit: robot biped_s52, 48 links, 47 joints
Links:
- link waist_yaw_link: mass 16.28826 -> 19.54016

File: src/kuavo_assets/models/biped_s52/urdf/drake/biped_v3.urdf (robot description, URDF)
Before this commit: robot biped_v3, 14 links, 13 joints
Links:
- link waist_yaw_link: mass 29.19556 -> 32.44746

File: src/kuavo_assets/models/biped_s52/urdf/drake/biped_v3_all_joint.urdf (robot description, URDF)
Before this commit: robot biped_v3_all_joint, 35 links, 30 joints
Links:
- link torso: mass 34.07404316 -> 37.32594316

File: src/kuavo_assets/models/biped_s52/urdf/drake/biped_v3_full.urdf (robot description, URDF)
Before this commit: robot biped_s52, 32 links, 31 joints
Links:
- link waist_yaw_link: mass 18.21145568 -> 21.46335568
