Commit message: 任务一传统方案初始实现

File: src/challenge_cup_simulator/models/biped_s52/urdf/drake/biped_v3_arm.urdf (robot description, URDF)
Before this commit: robot biped_s52, 18 links, 17 joints
Joints:
- joint zarm_l7_end_effector_joint: origin xyz=0 -0.03 -0.12 rpy=0 0 0 -> xyz=0 0 -0.1488 rpy=0 0 0
- joint zarm_r7_end_effector_joint: origin xyz=0 0.03 -0.12 rpy=0 0 0 -> xyz=0 0 -0.1488 rpy=0 0 0
